Commit message: Bug fix: 使用 Gazebo Harmonic (gz-sim 8.x), 解决 collision meshes导致的问题,解决 no clock 的问题,使用 xacro 使用 Gazebo Harmonic plugin

File: hunter_description/description/meshes.xacro (robot description, xacro)
@@ -8,10 +8,4 @@
       </geometry>
     </visual>
-    <collision>
-      <origin xyz="0 0 0" rpy="0 0 0"/>
-      <geometry>
-        <mesh filename="file://$(find hunter_description)/meshes/${name}.dae" />
-      </geometry>
-    </collision>
   </xacro:macro>
   <xacro:macro name="virtual">

File: hunter_description/description/robot_core.xacro (robot description, xacro)
@@ -18,8 +18,20 @@
   <link name="chassis">
     <xacro:mesh name="chassis"/>
+    <collision>
+      <origin xyz="0 0 0" rpy="0 0 0"/>
+      <geometry>
+        <box size="0.80 0.55 0.25"/>
+      </geometry>
+    </collision>
     <xacro:inertial_chassis/>
   </link>
   <link name="rear_left_wheel">
     <xacro:mesh name="rear_left_wheel"/>
+    <collision>
+      <origin xyz="0 0 0" rpy="${pi/2} 0 0"/>
+      <geometry>
+        <cylinder radius="0.165" length="0.10"/>
+      </geometry>
+    </collision>
     <xacro:inertial_wheel/>
   </link>
@@ -35,4 +47,10 @@
   <link name="rear_right_wheel">
     <xacro:mesh name="rear_right_wheel"/>
+    <collision>
+      <origin xyz="0 0 0" rpy="${pi/2} 0 0"/>
+      <geometry>
+        <cylinder radius="0.165" length="0.10"/>
+      </geometry>
+    </collision>
     <xacro:inertial_wheel/>
   </link>
@@ -61,4 +79,10 @@
   <link name="front_left_wheel">
     <xacro:mesh name="front_left_wheel"/>
+    <collision>
+      <origin xyz="0 0 0" rpy="${pi/2} 0 0"/>
+      <geometry>
+        <cylinder radius="0.165" length="0.10"/>
+      </geometry>
+    </collision>
     <xacro:inertial_wheel/>
   </link>
@@ -84,4 +108,10 @@
   <link name="front_right_wheel">
     <xacro:mesh name="front_right_wheel"/>
+    <collision>
+      <origin xyz="0 0 0" rpy="${pi/2} 0 0"/>
+      <geometry>
+        <cylinder radius="0.165" length="0.10"/>
+      </geometry>
+    </collision>
     <xacro:inertial_wheel/>
   </link>

File: hunter_description/description/robot_core_real_hack.xacro (robot description, xacro)
@@ -18,8 +18,20 @@
   <link name="chassis">
     <xacro:mesh name="chassis"/>
+    <collision>
+      <origin xyz="0 0 0" rpy="0 0 0"/>
+      <geometry>
+        <box size="0.80 0.55 0.25"/>
+      </geometry>
+    </collision>
     <xacro:inertial_chassis/>
   </link>
   <link name="rear_left_wheel">
     <xacro:mesh name="rear_left_wheel"/>
+    <collision>
+      <origin xyz="0 0 0" rpy="${pi/2} 0 0"/>
+      <geometry>
+        <cylinder radius="0.165" length="0.10"/>
+      </geometry>
+    </collision>
     <xacro:inertial_wheel/>
   </link>
@@ -35,4 +47,10 @@
   <link name="rear_right_wheel">
     <xacro:mesh name="rear_right_wheel"/>
+    <collision>
+      <origin xyz="0 0 0" rpy="${pi/2} 0 0"/>
+      <geometry>
+        <cylinder radius="0.165" length="0.10"/>
+      </geometry>
+    </collision>
     <xacro:inertial_wheel/>
   </link>
@@ -61,4 +79,10 @@
   <link name="front_left_wheel">
     <xacro:mesh name="front_left_wheel"/>
+    <collision>
+      <origin xyz="0 0 0" rpy="${pi/2} 0 0"/>
+      <geometry>
+        <cylinder radius="0.165" length="0.10"/>
+      </geometry>
+    </collision>
     <xacro:inertial_wheel/>
   </link>
@@ -85,4 +109,10 @@
   <link name="front_right_wheel">
     <xacro:mesh name="front_right_wheel"/>
+    <collision>
+      <origin xyz="0 0 0" rpy="${pi/2} 0 0"/>
+      <geometry>
+        <cylinder radius="0.165" length="0.10"/>
+      </geometry>
+    </collision>
     <xacro:inertial_wheel/>
   </link>

File: hunter_description/description/ros2_control.xacro (robot description, xacro)
@@ -3,5 +3,5 @@
   <ros2_control name="GazeboSystem" type="system">
     <hardware>
-      <plugin>gazebo_ros2_control/GazeboSystem</plugin>
+      <plugin>gz_ros2_control/GazeboSimSystem</plugin>
     </hardware>
     <joint name="front_left_steering_joint">
@@ -10,6 +10,5 @@
     </joint>
     <joint name="front_right_steering_joint">
-      <param name="mimic">front_left_steering_joint</param>
-      <param name="multiplier">1</param>
+      <mimic joint="front_left_steering_joint" multiplier="1" />
       <state_interface name="position"/>
     </joint>
@@ -20,6 +19,5 @@
     </joint>
     <joint name="rear_right_wheel_joint">
-      <param name="mimic">rear_left_wheel_joint</param>
-      <param name="multiplier">1</param>
+      <mimic joint="rear_left_wheel_joint" multiplier="1" />
       <state_interface name="velocity"/>
       <state_interface name="position"/>
@@ -35,5 +33,5 @@
   </ros2_control>
   <gazebo>
-    <plugin filename="libgazebo_ros2_control.so" name="gazebo_ros2_control">
+    <plugin filename="libgz_ros2_control-system.so" name="gz_ros2_control::GazeboSimROS2ControlPlugin">
       <parameters>$(find hunter_description)/config/ackermann_like_controller.yaml</parameters>
     </plugin>
