Commit message: 移植到新版GZ SIM,使用ros2_control作为控制

File: hunter_description/description/inertial_macros.xacro (robot description, xacro)
@@ -1,18 +1,9 @@
 <?xml version="1.0"?>
-<robot xmlns:xacro="http://www.ros.org/wiki/xacro" >
+<robot xmlns:xacro="http://www.ros.org/wiki/xacro">
   <xacro:macro name="inertial_chassis">
     <inertial>
-      <origin
-        xyz="0.0266989327622036 0.000409203500587652 -0.135901124750884"
-        rpy="0 0 0" />
-      <mass
-        value="72" />
-      <inertia
-        ixx="0.0332370959804736"
-        ixy="-1.013150489971E-06"
-        ixz="-0.00188859201421112"
-        iyy="0.111072002332437"
-        iyz="-5.13308150598312E-07"
-        izz="0.12660862809283" />
+      <origin rpy="0 0 0" xyz="0 0 0" />
+      <mass value="72" />
+      <inertia ixx="2.02" ixy="0.0" ixz="0.0" iyy="4.03" iyz="0.0" izz="5.11" />
     </inertial>
   </xacro:macro>
@@ -34,17 +25,9 @@
   </xacro:macro>
   <xacro:macro name="inertial_steering_link">
+    <!-- 修改惯量参数否则关节非常难带动,看起来像卡住。 -->
     <inertial>
-      <origin
-        xyz="0 0 0"
-        rpy="0 0 0" />
-      <mass
-        value="0.005" />
-      <inertia
-        ixx="0.1"
-        ixy="0"
-        ixz="0"
-        iyy="0.1"
-        iyz="0"
-        izz="0.1" />
+      <origin rpy="0 0 0" xyz="0 0 0" />
+      <mass value="0.1" />
+      <inertia ixx="1e-4" ixy="0" ixz="0" iyy="1e-4" iyz="0" izz="1e-4" />
     </inertial>
   </xacro:macro>

File: hunter_description/description/meshes.xacro (robot description, xacro)
@@ -22,9 +22,10 @@
   <xacro:macro name="gazebo_friction" params="reference">
     <gazebo reference="${reference}">
-      <mu1 value="1.0"/>
-      <mu2 value="0.5"/>
-      <kp value="10000000.0" />
+      <mu1 value="0.6"/>
+      <mu2 value="0.6"/>
+      <!-- 接触刚性太高,小车会弹起来。 -->
+      <!-- <kp value="10000000.0" />
       <kd value="1.0" />
-      <fdir1 value="1 0 0"/>
+      <fdir1 value="1 0 0"/> -->
     </gazebo>
   </xacro:macro>

File: hunter_description/description/robot_core.xacro (robot description, xacro)
@@ -19,7 +19,7 @@
     <xacro:mesh name="chassis"/>
     <collision>
-      <origin xyz="0 0 0" rpy="0 0 0"/>
+      <origin xyz="0 0 -0.12" rpy="0 0 0"/>
       <geometry>
-        <box size="0.80 0.55 0.25"/>
+        <box size="0.85 0.3 0.25"/>
       </geometry>
     </collision>
@@ -29,5 +29,5 @@
     <xacro:mesh name="rear_left_wheel"/>
     <collision>
-      <origin xyz="0 0 0" rpy="${pi/2} 0 0"/>
+      <origin xyz="0 0 0" rpy="0 0 0"/>
       <geometry>
         <cylinder radius="0.165" length="0.10"/>
@@ -41,6 +41,7 @@
     <origin xyz="${x_base_to_rear} ${y_base_to_wheel} ${z_base_to_wheel}" rpy="${pi/2} 0 0" />
     <axis xyz="0 0 -1" />
-    <dynamics damping="0.2" friction="15"/>
-    <limit effort="10.0" velocity="10.0"/>
+    <!-- 阻力不可以太大否则根本转不动 -->
+    <dynamics damping="0.05" friction="0.0"/>
+    <limit effort="100.0" velocity="30.0"/>
   </joint>
   <xacro:gazebo_friction reference="rear_left_wheel"/>
@@ -48,5 +49,5 @@
     <xacro:mesh name="rear_right_wheel"/>
     <collision>
-      <origin xyz="0 0 0" rpy="${pi/2} 0 0"/>
+      <origin xyz="0 0 0" rpy="0 0 0"/>
       <geometry>
         <cylinder radius="0.165" length="0.10"/>
@@ -60,7 +61,7 @@
     <origin xyz="${x_base_to_rear} -${y_base_to_wheel} ${z_base_to_wheel}" rpy="${pi/2} 0 0" />
     <axis xyz="0 0 -1"/>
-    <dynamics damping="0.2" friction="15"/>
-    <limit effort="10.0" velocity="10.0"/>
-    <mimic joint="rear_left_wheel_joint" multiplier="1.0" offset="0.0"/>
+    <!-- 阻力不可以太大否则根本转不动 -->
+    <dynamics damping="0.05" friction="0.0"/>
+    <limit effort="100.0" velocity="30.0"/>
   </joint>
   <xacro:gazebo_friction reference="rear_right_wheel"/>
@@ -74,11 +75,11 @@
     <origin xyz="${x_base_to_front} ${y_base_to_wheel} ${z_base_to_wheel}" rpy="${pi/2} 0 0" />
     <axis   xyz="0 1 0" />
-    <limit  lower="-${max_steer_angle_central}"  upper="${max_steer_angle_central}"  effort="10.0"  velocity="1" />
-    <dynamics damping="0.2"/>
+    <limit  lower="-${max_steer_angle_central}"  upper="${max_steer_angle_central}"  effort="100.0"  velocity="2.0" />
+    <dynamics damping="0.5" friction="0.0"/>
   </joint>
   <link name="front_left_wheel">
     <xacro:mesh name="front_left_wheel"/>
     <collision>
-      <origin xyz="0 0 0" rpy="${pi/2} 0 0"/>
+      <origin xyz="0 0 0" rpy="0 0 0"/>
       <geometry>
         <cylinder radius="0.165" length="0.10"/>
@@ -93,4 +94,6 @@
     <axis   xyz="0 0 -1" />
   </joint>
+  <!-- 需要给前轮也补充摩擦系数 -->
+  <xacro:gazebo_friction reference="front_left_wheel"/>
   <link name="front_right_steering_link">
     <xacro:virtual/>
@@ -102,12 +105,11 @@
     <origin xyz="${x_base_to_front}  -${y_base_to_wheel} ${z_base_to_wheel}" rpy="${pi/2} 0 0" />
     <axis   xyz="0 1 0" />
-    <limit  lower="-${max_steer_angle_central}"  upper="${max_steer_angle_central}"  effort="10.0"  velocity="1" />
-    <dynamics damping="0.2"/>
-    <mimic joint="front_left_steering_joint" multiplier="1.0" offset="0.0"/>
+    <limit  lower="-${max_steer_angle_central}"  upper="${max_steer_angle_central}"  effort="100.0"  velocity="2.0" />
+    <dynamics damping="0.5" friction="0.0"/>
   </joint>
   <link name="front_right_wheel">
     <xacro:mesh name="front_right_wheel"/>
     <collision>
-      <origin xyz="0 0 0" rpy="${pi/2} 0 0"/>
+      <origin xyz="0 0 0" rpy="0 0 0"/>
       <geometry>
         <cylinder radius="0.165" length="0.10"/>
@@ -122,3 +124,5 @@
     <axis   xyz="0 0 -1" />
   </joint>
+  <!-- 需要给前轮也补充摩擦系数 -->
+  <xacro:gazebo_friction reference="front_right_wheel"/>
 </robot>

File: hunter_description/description/ros2_control.xacro (robot description, xacro)
@@ -1,4 +1,5 @@
 <?xml version="1.0"?>
 <robot xmlns:xacro="http://www.ros.org/wiki/xacro">
+  <!-- 声明这些 joint 暴露哪些 command/state interfaces，以及它们属于哪个 hardware component -->
   <ros2_control name="GazeboSystem" type="system">
     <hardware>
@@ -10,5 +11,5 @@
     </joint>
     <joint name="front_right_steering_joint">
-      <mimic joint="front_left_steering_joint" multiplier="1" />
+      <command_interface name="position"/>
       <state_interface name="position"/>
     </joint>
@@ -19,5 +20,5 @@
     </joint>
     <joint name="rear_right_wheel_joint">
-      <mimic joint="rear_left_wheel_joint" multiplier="1" />
+      <command_interface name="velocity"/>
       <state_interface name="velocity"/>
       <state_interface name="position"/>
@@ -32,4 +33,5 @@
     </joint>
   </ros2_control>
+  <!-- 在 Gazebo 启动时实例化 controller_manager，并把 Gazebo model 接到 ros2_control -->
   <gazebo>
     <plugin filename="libgz_ros2_control-system.so" name="gz_ros2_control::GazeboSimROS2ControlPlugin">
